File: _autosave-Power-Distribution-Board.kicad_pcb (KiCad board)
At the start: 2 copper layers, 12 parts, among them J1 XT60PB-F, J10 XT30UPB-F, J11 XT30UPB-F, J12 XT90PB-F, J2 XT30UPB-F, J3 XT30UPB-F, J4 XT30UPB-F, J5 XT30UPB-F, J6 XT30UPB-F, J7 XT30UPB-F, J8 XT30UPB-F, J9 XT30UPB-F

Commit message: pressed B
oh goodness
Routing:
- added copper zone on B.Cu, net (none)
Changed lines of the file:
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@@
 		(min_thickness 0.25)
 		(filled_areas_thickness no)
-		(fill
+		(fill yes
 			(thermal_gap 0.5)
 			(thermal_bridge_width 0.5)
@@
 			)
 		)
+	)
+	(zone
+		(net 0)
+		(net_name "")
+		(layer "B.Cu")
+		(hatch edge 0.5)
+		(priority 1)
+		(connect_pads
+			(clearance 0.5)
+		)
+		(min_thickness 0.25)
+		(filled_areas_thickness no)
+		(fill yes
+			(thermal_gap 0.5)
+			(thermal_bridge_width 0.5)
+			(island_removal_mode 1)
+			(island_area_min 10)
+		)
+		(polygon
+			(pts
+				(xy 163 56.25) (xy 191 56.5) (xy 190.5 125.5) (xy 163.25 125.5)
+			)
+		)
